File: stm32.sch (KiCad schematic (older format))
At the start: 43 parts, among them J1 USB_B_Micro, J2 Conn_02x05_Odd_Even, J3 Conn_01x02, SW1 SW_Push, SW2 SW_Push, U1 STM32F407VGT6, U5 LM1117-3.3, X1 8MHz 20pF, Y2 32768 Hz

Commit message: Replace micro USB connector with through hole version
Parts:
- J1: footprint Connector_USB:USB_Micro-B_Molex-105133-0031 -> Connectors_USB:USB_Micro-B_Wuerth-614105150721_Vertical; Manufacturer MOLEX -> GCT; Part # 105133-0031 -> USB3131-30-0230-A; VEND MOUSER -> DIGI; VEND# 538-105133-0031 -> 2073-USB3131-30-0230-ACT-ND
Changed lines of the file:
@@
 EESchema Schematic File Version 4
 LIBS:microRusEfi-cache
-EELAYER 29 0
+EELAYER 30 0
 EELAYER END
 $Descr B 17000 11000
@@
 F 0 "J1" H 11557 4667 50  0000 C CNN
 F 1 "USB_B_Micro" H 11557 4576 50  0000 C CNN
-F 2 "Connector_USB:USB_Micro-B_Molex-105133-0031" H 11650 4150 50  0001 C CNN
+F 2 "Connectors_USB:USB_Micro-B_Wuerth-614105150721_Vertical" H 11650 4150 50  0001 C CNN
 F 3 "~" H 11650 4150 50  0001 C CNN
-F 4 "MOLEX" H 0   0   50  0001 C CNN "Manufacturer"
-F 5 "105133-0031" H 0   0   50  0001 C CNN "Part #"
-F 6 "MOUSER" H 0   0   50  0001 C CNN "VEND"
-F 7 "538-105133-0031" H 0   0   50  0001 C CNN "VEND#"
+F 4 "GCT" H 0   0   50  0001 C CNN "Manufacturer"
+F 5 "USB3131-30-0230-A" H 0   0   50  0001 C CNN "Part #"
+F 6 "DIGI" H 0   0   50  0001 C CNN "VEND"
+F 7 "2073-USB3131-30-0230-ACT-ND" H 0   0   50  0001 C CNN "VEND#"
 	1    11500 4200
 	1    0    0    -1

Commit message: Fix mixed up AV4, AV5, 5Vsense, and 12V sense
Parts:
- D19: Manufacturer (none) -> Lite-On
Changed lines of the file:
@@
 F 3 "" H 15400 3400 60  0000 C CNN
 F 4 "C2286" H 15400 3400 50  0001 C CNN "LCSC"
+F 5 "Lite-On " H 15400 3400 50  0001 C CNN "Manufacturer"
 	1    15400 3400
 	-1   0    0    1
